File: B0_14CN3801.sch (EAGLE design)
At the start: 1 part

Commit message: .
Parts:
- added C1, C2: 100n, rcl:C-EUC0805
- added C4: 220n, rcl:C-EUC0805
- added HL1, HL2: (no value), led:LEDCHIPLED_0603
- added JP1: (no value), Разъёмы штырьковые 2.54мм:PINHD-1X2/2
- added R1, R3, R4: (no value), rcl:R-EU_R0805
- added R2: 120, rcl:R-EU_R0805
- added VT1: (no value), m_transistor:MOSFET-P_TO220_V
- renumbered DA14 to DA1
Connections:
- new net GND: C1.2, C4.2, DA1.GND, JP1.2, R4.1
- new net N$1: C1.1, C2.1, DA1.VCC, JP1.1, R1.2, R3.2, VT1.S
- new net N$2: C2.2, DA1.VG
- new net N$3: DA1.MPPT, R3.1, R4.2
- new net N$4: DA1.COM, R2.2
- new net N$5: HL1.A, HL2.A, R1.1
- new net N$6: DA1.!CHRG, HL1.C
- new net N$7: DA1.!DONE, HL2.C
- new net N$8: C4.1, R2.1
- new net N$9: DA1.DRV, VT1.G

Commit message: .
Parts:
- added C1B, C3B: 1mf cer, rcl:C-EUC0805
- added C1C: 47m, rcl:CPOL-EUE2.5-6
- added C3: 10m louesr, rcl:CPOL-EUE2.5-6
Connections:
- new net N$10: C3.+, C3B.1
- net GND: now also C3.-, C3B.2
Other:
- note added: "1.205v max"
- moved on the sheet: C1, JP1, R3, R4

Commit message: .
Parts:
- added D1, D2, D3: (no value), diode:SCHOTTKY-DIODESMC
Changed lines of the file:
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@@
 <part name="C3B" library="rcl" deviceset="C-EU" device="C0805" value="1mf cer"/>
 <part name="GND7" library="supply1v" deviceset="GND" device=""/>
+<part name="D1" library="diode" deviceset="SCHOTTKY-DIODE" device="SMC"/>
+<part name="D2" library="diode" deviceset="SCHOTTKY-DIODE" device="SMC"/>
+<part name="D3" library="diode" deviceset="SCHOTTKY-DIODE" device="SMC"/>
 </parts>
 <sheets>
@@
 </instance>
 <instance part="GND7" gate="1" x="83.82" y="53.34"/>
+<instance part="D1" gate="G$1" x="-35.56" y="93.98"/>
+<instance part="D2" gate="G$1" x="-35.56" y="83.82"/>
+<instance part="D3" gate="G$1" x="-35.56" y="88.9"/>
 </instances>
 <busses>

Commit message: .
Other:
- moved on the sheet: C4, R2
Changed lines of the file:
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@@
 <part name="C1" library="rcl" deviceset="C-EU" device="C0805" value="100n"/>
 <part name="GND1" library="supply1v" deviceset="GND" device=""/>
-<part name="GND2" library="supply1v" deviceset="GND" device=""/>
 <part name="HL1" library="led" deviceset="LED" device="CHIPLED_0603"/>
 <part name="HL2" library="led" deviceset="LED" device="CHIPLED_0603"/>
@@
 </instance>
 <instance part="GND1" gate="1" x="-12.7" y="53.34"/>
-<instance part="GND2" gate="1" x="50.8" y="35.56"/>
 <instance part="HL1" gate="G$1" x="10.16" y="50.8" smashed="yes" rot="R90">
 <attribute name="NAME" x="12.192" y="54.356" size="1.778" layer="95" rot="R180"/>
@@
 <attribute name="VALUE" x="5.842" y="57.15" size="1.778" layer="96" rot="R90"/>
 </instance>
-<instance part="R2" gate="G$1" x="58.42" y="38.1" smashed="yes" rot="R90">
-<attribute name="NAME" x="59.69" y="39.5986" size="1.778" layer="95"/>
-<attribute name="VALUE" x="59.69" y="37.338" size="1.778" layer="96"/>
+<instance part="R2" gate="G$1" x="60.96" y="38.1" smashed="yes" rot="R90">
+<attribute name="NAME" x="62.23" y="39.5986" size="1.778" layer="95"/>
+<attribute name="VALUE" x="62.23" y="37.338" size="1.778" layer="96"/>
 </instance>
 <instance part="R3" gate="G$1" x="-5.08" y="53.34" smashed="yes" rot="R90">
@@
 </instance>
 <instance part="GND3" gate="1" x="-5.08" y="22.86"/>
-<instance part="C4" gate="G$1" x="58.42" y="27.94"/>
-<instance part="GND4" gate="1" x="58.42" y="17.78"/>
+<instance part="C4" gate="G$1" x="60.96" y="27.94"/>
+<instance part="GND4" gate="1" x="50.8" y="33.02"/>
 <instance part="VT1" gate="G$1" x="53.34" y="66.04" smashed="yes" rot="R90">
 <attribute name="NAME" x="50.8" y="71.12" size="1.778" layer="95"/>
@@
 <net name="GND" class="0">
 <segment>
-<pinref part="DA1" gate="DA" pin="GND"/>
-<wire x1="48.26" y1="40.64" x2="50.8" y2="40.64" width="0.1524" layer="91"/>
-<pinref part="GND2" gate="1" pin="GND"/>
-<wire x1="50.8" y1="40.64" x2="50.8" y2="38.1" width="0.1524" layer="91"/>
-</segment>
-<segment>
 <pinref part="C1" gate="G$1" pin="2"/>
 <pinref part="GND1" gate="1" pin="GND"/>
@@
 <pinref part="C4" gate="G$1" pin="2"/>
 <pinref part="GND4" gate="1" pin="GND"/>
-<wire x1="58.42" y1="22.86" x2="58.42" y2="20.32" width="0.1524" layer="91"/>
+<wire x1="55.88" y1="20.32" x2="55.88" y2="40.64" width="0.1524" layer="91"/>
+<pinref part="DA1" gate="DA" pin="GND"/>
+<wire x1="55.88" y1="40.64" x2="50.8" y2="40.64" width="0.1524" layer="91"/>
+<wire x1="50.8" y1="40.64" x2="48.26" y2="40.64" width="0.1524" layer="91"/>
+<wire x1="50.8" y1="35.56" x2="50.8" y2="40.64" width="0.1524" layer="91"/>
+<wire x1="55.88" y1="20.32" x2="60.96" y2="20.32" width="0.1524" layer="91"/>
+<wire x1="60.96" y1="20.32" x2="60.96" y2="22.86" width="0.1524" layer="91"/>
+<junction x="50.8" y="40.64"/>
 </segment>
 <segment>
@@
 <segment>
 <pinref part="DA1" gate="DA" pin="COM"/>
-<wire x1="48.26" y1="45.72" x2="58.42" y2="45.72" width="0.1524" layer="91"/>
+<wire x1="48.26" y1="45.72" x2="60.96" y2="45.72" width="0.1524" layer="91"/>
 <pinref part="R2" gate="G$1" pin="2"/>
-<wire x1="58.42" y1="45.72" x2="58.42" y2="43.18" width="0.1524" layer="91"/>
+<wire x1="60.96" y1="45.72" x2="60.96" y2="43.18" width="0.1524" layer="91"/>
 </segment>
 </net>
@@
 <segment>
 <pinref part="R2" gate="G$1" pin="1"/>
-<wire x1="58.42" y1="33.02" x2="58.42" y2="30.48" width="0.1524" layer="91"/>
+<wire x1="60.96" y1="33.02" x2="60.96" y2="30.48" width="0.1524" layer="91"/>
 <pinref part="C4" gate="G$1" pin="1"/>
 </segment>

Commit message: .
Parts:
- added L1: (no value), rcl:L-USPIS2816
- added L2: (no value), rcl:L-USWE-TPC
- added L3: DR125, inductors:DR125
- added L4: DR127, inductors:DR127
Connections:
- net N$4 renamed COM
Changed lines of the file:
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@@
 <part name="D2" library="diode" deviceset="SCHOTTKY-DIODE" device="SMC"/>
 <part name="D3" library="diode" deviceset="SCHOTTKY-DIODE" device="SMC"/>
+<part name="L1" library="rcl" deviceset="L-US" device="PIS2816"/>
+<part name="L2" library="rcl" deviceset="L-US" device="WE-TPC"/>
+<part name="L3" library="inductors" deviceset="DR125" device=""/>
+<part name="L4" library="inductors" deviceset="DR127" device=""/>
 </parts>
 <sheets>
@@
 <instance part="D2" gate="G$1" x="-35.56" y="83.82"/>
 <instance part="D3" gate="G$1" x="-35.56" y="88.9"/>
+<instance part="L1" gate="G$1" x="20.32" y="12.7"/>
+<instance part="L2" gate="G$1" x="33.02" y="12.7"/>
+<instance part="L3" gate="G$1" x="53.34" y="7.62"/>
+<instance part="L4" gate="G$1" x="53.34" y="-2.54"/>
 </instances>
 <busses>
@@
 </segment>
 </net>
-<net name="N$4" class="0">
+<net name="COM" class="0">
 <segment>
 <pinref part="DA1" gate="DA" pin="COM"/>

Commit message: .
Parts:
- removed L1: (no value), rcl:L-USPIS2816
- removed L2: (no value), rcl:L-USWE-TPC
- removed L4: DR127, inductors:DR127
- removed VT1: (no value), m_transistor:MOSFET-P_TO220_V
- added D4, D5, D6: (no value), diode:SCHOTTKY-DIODESMC
- added Q1, Q4: BSO201SP, transistor-fet:BSO201SP
- added Q2, Q3: BSS84, transistor-fet:BSA223SP
- added R5: 332k, rcl:R-EU_R0805
- added RSC: (no value), rcl:R-EU_R0805
- added SJ1, SJ2: (no value), jumper:SJ
- R3: value (none) -> 43k
- R4: value (none) -> 15k
Connections:
- removed net N$10: C3.+, C3B.1
- new net BAT: DA1.BAT, Q3.D, SJ2.1
- new net CSP: DA1.CSP, Q2.D, SJ1.1
- new net N$11: L3.2, Q4.D
- new net N$12: Q2.G, Q3.G, Q4.G, R5.1
- new net N$13: D1.C, D3.C, D4.C, L3.1, Q1.D
- new net N$14: Q2.S, Q4.S, RSC.2, SJ1.2
- new net N$15: C3.+, C3B.1, Q3.S, R5.2, RSC.1, SJ2.2
- new net N$4: D2.A, D5.A, D6.A, JP1.1
- net GND: now also D1.A, D3.A, D4.A
- net N$1: now also D2.C, D5.C, D6.C, Q1.S; no longer JP1.1, VT1.S
- net N$9: now also Q1.G; no longer VT1.G
Other:
- moved on the sheet: C3, C3B, C4, D1, D2, D3, JP1, L3, R2

Commit message: .
Connections:
- net GND: now also C1B.2, C1C.-
- net N$1: now also C1B.1, C1C.+
Other:
- moved on the sheet: C3, C3B, RSC
Changed lines of the file:
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@@
 <attribute name="VALUE" x="-11.176" y="63.881" size="1.778" layer="96"/>
 </instance>
-<instance part="GND1" gate="1" x="-12.7" y="53.34"/>
+<instance part="GND1" gate="1" x="-20.32" y="48.26"/>
 <instance part="HL1" gate="G$1" x="10.16" y="50.8" smashed="yes" rot="R90">
 <attribute name="NAME" x="12.192" y="54.356" size="1.778" layer="95" rot="R180"/>
@@
 </instance>
 <instance part="C1C" gate="G$1" x="-27.94" y="63.5"/>
-<instance part="C3" gate="G$1" x="119.38" y="43.18"/>
-<instance part="GND6" gate="1" x="119.38" y="33.02"/>
-<instance part="C3B" gate="G$1" x="132.08" y="43.18" smashed="yes">
-<attribute name="NAME" x="133.604" y="46.101" size="1.778" layer="95"/>
-<attribute name="VALUE" x="133.604" y="43.561" size="1.778" layer="96"/>
-</instance>
-<instance part="GND7" gate="1" x="132.08" y="33.02"/>
+<instance part="C3" gate="G$1" x="119.38" y="45.72"/>
+<instance part="GND6" gate="1" x="119.38" y="35.56"/>
+<instance part="C3B" gate="G$1" x="132.08" y="45.72" smashed="yes">
+<attribute name="NAME" x="133.604" y="48.641" size="1.778" layer="95"/>
+<attribute name="VALUE" x="133.604" y="46.101" size="1.778" layer="96"/>
+</instance>
+<instance part="GND7" gate="1" x="132.08" y="35.56"/>
 <instance part="D2" gate="G$1" x="-38.1" y="73.66"/>
 <instance part="L3" gate="G$1" x="81.28" y="73.66"/>
@@
 <attribute name="NAME" x="97.79" y="80.01" size="1.778" layer="95" rot="MR0"/>
 </instance>
-<instance part="RSC" gate="G$1" x="119.38" y="58.42" smashed="yes" rot="R90">
-<attribute name="NAME" x="123.4186" y="67.31" size="1.778" layer="95" rot="R270"/>
-<attribute name="VALUE" x="122.682" y="54.61" size="1.778" layer="96" rot="R90"/>
+<instance part="RSC" gate="G$1" x="119.38" y="60.96" smashed="yes" rot="R90">
+<attribute name="NAME" x="123.4186" y="69.85" size="1.778" layer="95" rot="R270"/>
+<attribute name="VALUE" x="122.682" y="57.15" size="1.778" layer="96" rot="R90"/>
 </instance>
 <instance part="R5" gate="G$1" x="106.68" y="43.18" smashed="yes">
@@
 <pinref part="C1" gate="G$1" pin="2"/>
 <pinref part="GND1" gate="1" pin="GND"/>
-<wire x1="-12.7" y1="58.42" x2="-12.7" y2="55.88" width="0.1524" layer="91"/>
+<wire x1="-20.32" y1="50.8" x2="-20.32" y2="53.34" width="0.1524" layer="91"/>
+<wire x1="-20.32" y1="53.34" x2="-12.7" y2="53.34" width="0.1524" layer="91"/>
+<wire x1="-12.7" y1="53.34" x2="-12.7" y2="58.42" width="0.1524" layer="91"/>
+<pinref part="C1B" gate="G$1" pin="2"/>
+<wire x1="-20.32" y1="58.42" x2="-20.32" y2="53.34" width="0.1524" layer="91"/>
+<wire x1="-20.32" y1="53.34" x2="-27.94" y2="53.34" width="0.1524" layer="91"/>
+<pinref part="C1C" gate="G$1" pin="-"/>
+<wire x1="-27.94" y1="53.34" x2="-27.94" y2="58.42" width="0.1524" layer="91"/>
+<junction x="-20.32" y="53.34"/>
 </segment>
 <segment>
@@
 <pinref part="C3B" gate="G$1" pin="2"/>
 <pinref part="GND7" gate="1" pin="GND"/>
-<wire x1="132.08" y1="38.1" x2="132.08" y2="35.56" width="0.1524" layer="91"/>
+<wire x1="132.08" y1="40.64" x2="132.08" y2="38.1" width="0.1524" layer="91"/>
 </segment>
 <segment>
 <pinref part="GND6" gate="1" pin="GND"/>
 <pinref part="C3" gate="G$1" pin="-"/>
-<wire x1="119.38" y1="35.56" x2="119.38" y2="38.1" width="0.1524" layer="91"/>
+<wire x1="119.38" y1="38.1" x2="119.38" y2="40.64" width="0.1524" layer="91"/>
 </segment>
 <segment>
@@
 <wire x1="-35.56" y1="73.66" x2="-33.02" y2="73.66" width="0.1524" layer="91"/>
 <pinref part="D5" gate="G$1" pin="C"/>
-<wire x1="-33.02" y1="73.66" x2="-12.7" y2="73.66" width="0.1524" layer="91"/>
+<wire x1="-33.02" y1="73.66" x2="-27.94" y2="73.66" width="0.1524" layer="91"/>
+<wire x1="-27.94" y1="73.66" x2="-20.32" y2="73.66" width="0.1524" layer="91"/>
+<wire x1="-20.32" y1="73.66" x2="-12.7" y2="73.66" width="0.1524" layer="91"/>
 <wire x1="-35.56" y1="68.58" x2="-33.02" y2="68.58" width="0.1524" layer="91"/>
 <wire x1="-33.02" y1="68.58" x2="-33.02" y2="73.66" width="0.1524" layer="91"/>
@@
 <junction x="-33.02" y="68.58"/>
 <junction x="-33.02" y="73.66"/>
+<pinref part="C1B" gate="G$1" pin="1"/>
+<wire x1="-20.32" y1="66.04" x2="-20.32" y2="73.66" width="0.1524" layer="91"/>
+<pinref part="C1C" gate="G$1" pin="+"/>
+<wire x1="-27.94" y1="66.04" x2="-27.94" y2="73.66" width="0.1524" layer="91"/>
+<junction x="-27.94" y="73.66"/>
+<junction x="-20.32" y="73.66"/>
 </segment>
 </net>
@@
 <junction x="104.14" y="73.66"/>
 <wire x1="93.98" y1="58.42" x2="91.44" y2="58.42" width="0.1524" layer="91"/>
-<wire x1="119.38" y1="63.5" x2="119.38" y2="73.66" width="0.1524" layer="91"/>
+<wire x1="119.38" y1="66.04" x2="119.38" y2="73.66" width="0.1524" layer="91"/>
 <wire x1="119.38" y1="73.66" x2="104.14" y2="73.66" width="0.1524" layer="91"/>
 <pinref part="SJ1" gate="1" pin="2"/>
@@
 <wire x1="76.2" y1="50.8" x2="114.3" y2="50.8" width="0.1524" layer="91"/>
 <wire x1="114.3" y1="50.8" x2="119.38" y2="50.8" width="0.1524" layer="91"/>
-<wire x1="119.38" y1="50.8" x2="119.38" y2="53.34" width="0.1524" layer="91"/>
+<wire x1="119.38" y1="50.8" x2="119.38" y2="55.88" width="0.1524" layer="91"/>
 <pinref part="RSC" gate="G$1" pin="1"/>
 <pinref part="C3" gate="G$1" pin="+"/>
-<wire x1="119.38" y1="45.72" x2="119.38" y2="48.26" width="0.1524" layer="91"/>
-<wire x1="119.38" y1="48.26" x2="132.08" y2="48.26" width="0.1524" layer="91"/>
+<wire x1="119.38" y1="48.26" x2="119.38" y2="50.8" width="0.1524" layer="91"/>
+<wire x1="119.38" y1="50.8" x2="132.08" y2="50.8" width="0.1524" layer="91"/>
 <pinref part="C3B" gate="G$1" pin="1"/>
-<wire x1="132.08" y1="48.26" x2="132.08" y2="45.72" width="0.1524" layer="91"/>
-<wire x1="132.08" y1="48.26" x2="144.78" y2="48.26" width="0.1524" layer="91"/>
-<junction x="132.08" y="48.26"/>
-<wire x1="119.38" y1="50.8" x2="119.38" y2="48.26" width="0.1524" layer="91"/>
+<wire x1="132.08" y1="50.8" x2="132.08" y2="48.26" width="0.1524" layer="91"/>
+<wire x1="132.08" y1="50.8" x2="144.78" y2="50.8" width="0.1524" layer="91"/>
+<junction x="132.08" y="50.8"/>
 <junction x="119.38" y="50.8"/>
-<junction x="119.38" y="48.26"/>
+<junction x="119.38" y="50.8"/>
 <pinref part="R5" gate="G$1" pin="2"/>
 <wire x1="111.76" y1="43.18" x2="114.3" y2="43.18" width="0.1524" layer="91"/>

Commit message: .
Other:
- moved on the sheet: C2, R3
Changed lines of the file:
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@@
 <instances>
 <instance part="DA1" gate="DA" x="33.02" y="50.8"/>
-<instance part="C2" gate="G$1" x="10.16" y="63.5"/>
+<instance part="C2" gate="G$1" x="10.16" y="66.04" smashed="yes">
+<attribute name="NAME" x="11.684" y="66.421" size="1.778" layer="95"/>
+<attribute name="VALUE" x="16.764" y="66.421" size="1.778" layer="96"/>
+</instance>
 <instance part="C1" gate="G$1" x="-12.7" y="63.5" smashed="yes">
-<attribute name="NAME" x="-11.176" y="66.421" size="1.778" layer="95"/>
-<attribute name="VALUE" x="-11.176" y="63.881" size="1.778" layer="96"/>
+<attribute name="NAME" x="-11.176" y="79.121" size="1.778" layer="95"/>
+<attribute name="VALUE" x="-11.176" y="76.581" size="1.778" layer="96"/>
 </instance>
 <instance part="GND1" gate="1" x="-20.32" y="48.26"/>
@@
 <attribute name="VALUE" x="57.15" y="37.338" size="1.778" layer="96"/>
 </instance>
-<instance part="R3" gate="G$1" x="-5.08" y="53.34" smashed="yes" rot="R90">
-<attribute name="NAME" x="-3.81" y="54.8386" size="1.778" layer="95"/>
-<attribute name="VALUE" x="-3.81" y="52.578" size="1.778" layer="96"/>
+<instance part="R3" gate="G$1" x="-5.08" y="55.88" smashed="yes" rot="R90">
+<attribute name="NAME" x="-3.81" y="57.3786" size="1.778" layer="95"/>
+<attribute name="VALUE" x="-3.81" y="55.118" size="1.778" layer="96"/>
 </instance>
 <instance part="R4" gate="G$1" x="-5.08" y="33.02" smashed="yes" rot="R90">
@@
 <instance part="GND5" gate="1" x="-50.8" y="50.8"/>
 <instance part="C1B" gate="G$1" x="-20.32" y="63.5" smashed="yes">
-<attribute name="NAME" x="-18.796" y="66.421" size="1.778" layer="95"/>
-<attribute name="VALUE" x="-18.796" y="63.881" size="1.778" layer="96"/>
-</instance>
-<instance part="C1C" gate="G$1" x="-27.94" y="63.5"/>
+<attribute name="NAME" x="-21.336" y="79.121" size="1.778" layer="95"/>
+<attribute name="VALUE" x="-21.336" y="76.581" size="1.778" layer="96"/>
+</instance>
+<instance part="C1C" gate="G$1" x="-27.94" y="63.5" smashed="yes">
+<attribute name="NAME" x="-29.337" y="79.2226" size="1.778" layer="95"/>
+<attribute name="VALUE" x="-29.337" y="76.6826" size="1.778" layer="96"/>
+</instance>
 <instance part="C3" gate="G$1" x="119.38" y="45.72"/>
 <instance part="GND6" gate="1" x="119.38" y="35.56"/>
@@
 </instance>
 <instance part="Q2" gate="G$1" x="86.36" y="55.88" smashed="yes" rot="MR90">
-<attribute name="VALUE" x="80.01" y="67.31" size="1.778" layer="96" rot="MR180"/>
-<attribute name="NAME" x="82.55" y="69.85" size="1.778" layer="95" rot="MR180"/>
+<attribute name="VALUE" x="90.17" y="54.61" size="1.778" layer="96" rot="MR180"/>
+<attribute name="NAME" x="92.71" y="57.15" size="1.778" layer="95" rot="MR180"/>
 </instance>
 <instance part="Q3" gate="G$1" x="68.58" y="48.26" smashed="yes" rot="MR90">
-<attribute name="VALUE" x="62.23" y="54.61" size="1.778" layer="96" rot="MR180"/>
-<attribute name="NAME" x="64.77" y="57.15" size="1.778" layer="95" rot="MR180"/>
+<attribute name="VALUE" x="74.93" y="46.99" size="1.778" layer="96" rot="MR180"/>
+<attribute name="NAME" x="77.47" y="49.53" size="1.778" layer="95" rot="MR180"/>
 </instance>
 <instance part="D4" gate="G$1" x="60.96" y="78.74" rot="R270"/>
@@
 <wire x1="17.78" y1="55.88" x2="10.16" y2="55.88" width="0.1524" layer="91"/>
 <pinref part="C2" gate="G$1" pin="2"/>
-<wire x1="10.16" y1="55.88" x2="10.16" y2="58.42" width="0.1524" layer="91"/>
+<wire x1="10.16" y1="55.88" x2="10.16" y2="60.96" width="0.1524" layer="91"/>
 </segment>
 </net>
@@
 <pinref part="R3" gate="G$1" pin="1"/>
 <pinref part="R4" gate="G$1" pin="2"/>
-<wire x1="-5.08" y1="48.26" x2="-5.08" y2="40.64" width="0.1524" layer="91"/>
+<wire x1="-5.08" y1="50.8" x2="-5.08" y2="40.64" width="0.1524" layer="91"/>
 <wire x1="-5.08" y1="40.64" x2="-5.08" y2="38.1" width="0.1524" layer="91"/>
 <pinref part="DA1" gate="DA" pin="MPPT"/>
@@
 <wire x1="15.24" y1="60.96" x2="15.24" y2="73.66" width="0.1524" layer="91"/>
 <pinref part="C2" gate="G$1" pin="1"/>
-<wire x1="10.16" y1="66.04" x2="10.16" y2="73.66" width="0.1524" layer="91"/>
+<wire x1="10.16" y1="68.58" x2="10.16" y2="73.66" width="0.1524" layer="91"/>
 <wire x1="10.16" y1="73.66" x2="15.24" y2="73.66" width="0.1524" layer="91"/>
 <wire x1="10.16" y1="73.66" x2="2.54" y2="73.66" width="0.1524" layer="91"/>
@@
 <wire x1="15.24" y1="73.66" x2="48.26" y2="73.66" width="0.1524" layer="91"/>
 <pinref part="R3" gate="G$1" pin="2"/>
-<wire x1="-5.08" y1="58.42" x2="-5.08" y2="73.66" width="0.1524" layer="91"/>
+<wire x1="-5.08" y1="60.96" x2="-5.08" y2="73.66" width="0.1524" layer="91"/>
 <junction x="-12.7" y="73.66"/>
 <junction x="-5.08" y="73.66"/>
