File: B0_14CN3801.sch (EAGLE design)
At the start: 30 parts, among them Q1 BSO201SP, Q2 BSS84, Q3 BSS84, Q4 BSO201SP

Commit message: t
Parts:
- added D10, D11, D12, D13, D14, D15, D16, D17, D18, D19, D20, D7, D8, D9: (no value), diode:SCHOTTKY-DIODESMC
- added JP10, JP11: (no value), Разъёмы штырьковые 2.54мм:PINHD-1X7
- added JP4: (no value), Разъёмы штырьковые 2.54мм:PINHD-2X7
- added JP8, JP9: (no value), Разъёмы штырьковые 2.54мм:PINHD-1X2/2
- added VT1, VT2: (no value), m_transistor:MOSFET-N_TO220_H
Connections:
- new net N$10: D14.C, D7.C
- new net N$16: D13.C, D15.C
- new net N$17: D12.C, D16.C
- new net N$18: D11.C, D17.C
- new net N$19: D10.C, D18.C
- new net N$20: D19.C, D9.C
- new net N$21: D20.C, D8.C
Other:
- note added: "SS36 3A 60v"
Changed lines of the file:
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@@
 <part name="SJ1" library="jumper" deviceset="SJ" device=""/>
 <part name="SJ2" library="jumper" deviceset="SJ" device=""/>
+<part name="JP4" library="Разъёмы штырьковые 2.54мм" deviceset="PINHD-2X7" device=""/>
+<part name="JP8" library="Разъёмы штырьковые 2.54мм" deviceset="PINHD-1X2" device="/2"/>
+<part name="JP9" library="Разъёмы штырьковые 2.54мм" deviceset="PINHD-1X2" device="/2"/>
+<part name="VT1" library="m_transistor" deviceset="MOSFET-N" device="_TO220_H"/>
+<part name="VT2" library="m_transistor" deviceset="MOSFET-N" device="_TO220_H"/>
+<part name="D8" library="diode" deviceset="SCHOTTKY-DIODE" device="SMC"/>
+<part name="D9" library="diode" deviceset="SCHOTTKY-DIODE" device="SMC"/>
+<part name="D10" library="diode" deviceset="SCHOTTKY-DIODE" device="SMC"/>
+<part name="D11" library="diode" deviceset="SCHOTTKY-DIODE" device="SMC"/>
+<part name="D12" library="diode" deviceset="SCHOTTKY-DIODE" device="SMC"/>
+<part name="D13" library="diode" deviceset="SCHOTTKY-DIODE" device="SMC"/>
+<part name="D14" library="diode" deviceset="SCHOTTKY-DIODE" device="SMC"/>
+<part name="D7" library="diode" deviceset="SCHOTTKY-DIODE" device="SMC"/>
+<part name="D15" library="diode" deviceset="SCHOTTKY-DIODE" device="SMC"/>
+<part name="D16" library="diode" deviceset="SCHOTTKY-DIODE" device="SMC"/>
+<part name="D17" library="diode" deviceset="SCHOTTKY-DIODE" device="SMC"/>
+<part name="D18" library="diode" deviceset="SCHOTTKY-DIODE" device="SMC"/>
+<part name="D19" library="diode" deviceset="SCHOTTKY-DIODE" device="SMC"/>
+<part name="D20" library="diode" deviceset="SCHOTTKY-DIODE" device="SMC"/>
+<part name="JP10" library="Разъёмы штырьковые 2.54мм" deviceset="PINHD-1X7" device=""/>
+<part name="JP11" library="Разъёмы штырьковые 2.54мм" deviceset="PINHD-1X7" device=""/>
 </parts>
 <sheets>
@@
 <plain>
 <text x="5.08" y="40.64" size="1.27" layer="98">1.205v max</text>
+<text x="-50.8" y="88.9" size="1.778" layer="91">SS36 3A 60v</text>
 </plain>
 <instances>
@@
 <instance part="SJ1" gate="1" x="86.36" y="63.5"/>
 <instance part="SJ2" gate="1" x="68.58" y="55.88"/>
+<instance part="JP4" gate="A" x="-93.98" y="7.62"/>
+<instance part="JP8" gate="G$1" x="-127" y="68.58"/>
+<instance part="JP9" gate="G$1" x="-111.76" y="68.58"/>
+<instance part="VT1" gate="G$1" x="-129.54" y="40.64"/>
+<instance part="VT2" gate="G$1" x="-129.54" y="27.94"/>
+<instance part="D8" gate="G$1" x="-162.56" y="7.62"/>
+<instance part="D9" gate="G$1" x="-162.56" y="2.54"/>
+<instance part="D10" gate="G$1" x="-162.56" y="-2.54"/>
+<instance part="D11" gate="G$1" x="-162.56" y="-7.62"/>
+<instance part="D12" gate="G$1" x="-162.56" y="-12.7"/>
+<instance part="D13" gate="G$1" x="-162.56" y="-17.78"/>
+<instance part="D14" gate="G$1" x="-162.56" y="-22.86"/>
+<instance part="D7" gate="G$1" x="-152.4" y="-22.86" rot="MR0"/>
+<instance part="D15" gate="G$1" x="-152.4" y="-17.78" rot="MR0"/>
+<instance part="D16" gate="G$1" x="-152.4" y="-12.7" rot="MR0"/>
+<instance part="D17" gate="G$1" x="-152.4" y="-7.62" rot="MR0"/>
+<instance part="D18" gate="G$1" x="-152.4" y="-2.54" rot="MR0"/>
+<instance part="D19" gate="G$1" x="-152.4" y="2.54" rot="MR0"/>
+<instance part="D20" gate="G$1" x="-152.4" y="7.62" rot="MR0"/>
+<instance part="JP10" gate="A" x="-71.12" y="38.1"/>
+<instance part="JP11" gate="A" x="-71.12" y="10.16"/>
 </instances>
 <busses>
@@
 </segment>
 </net>
+<net name="N$10" class="0">
+<segment>
+<pinref part="D14" gate="G$1" pin="C"/>
+<pinref part="D7" gate="G$1" pin="C"/>
+<wire x1="-154.94" y1="-22.86" x2="-160.02" y2="-22.86" width="0.1524" layer="91"/>
+</segment>
+</net>
+<net name="N$16" class="0">
+<segment>
+<pinref part="D13" gate="G$1" pin="C"/>
+<pinref part="D15" gate="G$1" pin="C"/>
+<wire x1="-154.94" y1="-17.78" x2="-160.02" y2="-17.78" width="0.1524" layer="91"/>
+</segment>
+</net>
+<net name="N$17" class="0">
+<segment>
+<pinref part="D12" gate="G$1" pin="C"/>
+<pinref part="D16" gate="G$1" pin="C"/>
+<wire x1="-154.94" y1="-12.7" x2="-160.02" y2="-12.7" width="0.1524" layer="91"/>
+</segment>
+</net>
+<net name="N$18" class="0">
+<segment>
+<pinref part="D11" gate="G$1" pin="C"/>
+<pinref part="D17" gate="G$1" pin="C"/>
+<wire x1="-154.94" y1="-7.62" x2="-160.02" y2="-7.62" width="0.1524" layer="91"/>
+</segment>
+</net>
+<net name="N$19" class="0">
+<segment>
+<pinref part="D10" gate="G$1" pin="C"/>
+<pinref part="D18" gate="G$1" pin="C"/>
+<wire x1="-154.94" y1="-2.54" x2="-160.02" y2="-2.54" width="0.1524" layer="91"/>
+</segment>
+</net>
+<net name="N$20" class="0">
+<segment>
+<pinref part="D9" gate="G$1" pin="C"/>
+<pinref part="D19" gate="G$1" pin="C"/>
+<wire x1="-154.94" y1="2.54" x2="-160.02" y2="2.54" width="0.1524" layer="91"/>
+</segment>
+</net>
+<net name="N$21" class="0">
+<segment>
+<pinref part="D8" gate="G$1" pin="C"/>
+<pinref part="D20" gate="G$1" pin="C"/>
+<wire x1="-154.94" y1="7.62" x2="-160.02" y2="7.62" width="0.1524" layer="91"/>
+</segment>
+</net>

Commit message: .
Parts:
- added JP2, JP3: (no value), Разъёмы штырьковые 2.54мм:PINHD-1X2/2
Connections:
- new net N$22: D19.A, JP3.2
- new net N$23: D9.A, JP3.1
- new net N$24: D8.A, JP2.1
- new net N$25: D20.A, JP2.2
- net N$10: now also JP11.7
- net N$16: now also JP11.6
- net N$17: now also JP11.5
- net N$18: now also JP11.4
- net N$19: now also JP11.3
- net N$20: now also JP11.2
- net N$21: now also JP11.1
Other:
- note added: "T1"
- moved on the sheet: D10, D11, D12, D13, D14, D15, D16, D17, D18, D19, D20, D7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
