File: B0_14CN3801.brd (EAGLE design)
At the start: 160 x 100 mm, 1 part

Commit message: .
Parts:
- added C1, C2: 100n, rcl:C0805
- added C4: 220n, rcl:C0805
- added HL1, HL2: (no value), led:CHIPLED_0603
- added JP1: (no value), Разъёмы штырьковые 2.54мм:1X02
- added R1, R3, R4: (no value), rcl:R0805
- added R2: 120, rcl:R0805
- added VT1: (no value), m_transistor:TO220FV
- renumbered DA14 to DA1
Connections:
- removed net VCC: DA1.9
- new net N$1: C1.1, C2.1, DA1.9, JP1.1, R1.2, R3.2, VT1.3
- new net N$2: C2.2, DA1.1
- new net N$3: DA1.6, R3.1, R4.2
- new net N$4: DA1.5, R2.2
- new net N$5: HL1.A, HL2.A, R1.1
- new net N$6: DA1.3, HL1.C
- new net N$7: DA1.4, HL2.C
- new net N$8: C4.1, R2.1
- new net N$9: DA1.10, VT1.1
- net GND: now also C1.2, C4.2, JP1.2, R4.1
Other:
- board outline removed

Commit message: .
Parts:
- added C1B, C3B: 1mf cer, rcl:C0805
- added C1C: 47m, rcl:E2,5-6
- added C3: 10m louesr, rcl:E2,5-6
Connections:
- new net N$10: C3.+, C3B.1
- net GND: now also C3.-, C3B.2
Changed lines of the file:
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@@
 <element name="VT1" library="m_transistor" package="TO220FV" value="" x="77.47" y="57.15" rot="R270"/>
 <element name="JP1" library="Разъёмы штырьковые 2.54мм" package="1X02" value="" x="57.15" y="61.595" rot="R270"/>
+<element name="C1B" library="rcl" package="C0805" value="1mf cer" x="45.085" y="38.1"/>
+<element name="C1C" library="rcl" package="E2,5-6" value="47m" x="45.72" y="31.75"/>
+<element name="C3" library="rcl" package="E2,5-6" value="10m louesr" x="45.72" y="24.765"/>
+<element name="C3B" library="rcl" package="C0805" value="1mf cer" x="45.085" y="18.415"/>
 </elements>
 <signals>
-<signal name="N$1">
-<contactref element="DA1" pad="9"/>
-<contactref element="C2" pad="1"/>
-<contactref element="C1" pad="1"/>
-<contactref element="R1" pad="2"/>
-<contactref element="R3" pad="2"/>
-<contactref element="VT1" pad="3"/>
-<contactref element="JP1" pad="1"/>
-<wire x1="67.31" y1="58.735" x2="67.63" y2="62.23" width="0" layer="19" extent="1-1"/>
-<wire x1="64.73" y1="59.42" x2="67.31" y2="58.735" width="0" layer="19" extent="1-1"/>
-<wire x1="59.69" y1="63.815" x2="64.73" y2="59.42" width="0" layer="19" extent="1-1"/>
-<wire x1="57.15" y1="62.865" x2="59.69" y2="63.815" width="0" layer="19" extent="1-1"/>
-<wire x1="54.61" y1="61.275" x2="57.15" y2="62.865" width="0" layer="19" extent="1-1"/>
-<wire x1="74.93" y1="54.61" x2="67.31" y2="58.735" width="0" layer="19" extent="1-1"/>
-</signal>
 <signal name="N$2">
 <contactref element="DA1" pad="1"/>
@@
 <contactref element="C4" pad="2"/>
 <contactref element="JP1" pad="2"/>
+<contactref element="C3B" pad="2"/>
+<contactref element="C3" pad="-"/>
 <wire x1="69.85" y1="60.005" x2="69.53" y2="62.23" width="0" layer="19" extent="1-1"/>
 <wire x1="65.72" y1="54.61" x2="69.85" y2="60.005" width="0" layer="19" extent="1-1"/>
 <wire x1="59.73" y1="59.42" x2="65.72" y2="54.61" width="0" layer="19" extent="1-1"/>
 <wire x1="57.15" y1="60.325" x2="59.73" y2="59.42" width="0" layer="19" extent="1-1"/>
+<wire x1="46.99" y1="24.765" x2="65.72" y2="54.61" width="0" layer="19" extent="1-1"/>
+<wire x1="46.035" y1="18.415" x2="46.99" y2="24.765" width="0" layer="19" extent="1-1"/>
 </signal>
 <signal name="N$5">
@@
 <wire x1="64.73" y1="60.42" x2="74.93" y2="59.69" width="0" layer="19" extent="1-1"/>
 </signal>
+<signal name="N$1">
+<contactref element="JP1" pad="1"/>
+<contactref element="DA1" pad="9"/>
+<contactref element="C2" pad="1"/>
+<contactref element="C1" pad="1"/>
+<contactref element="R1" pad="2"/>
+<contactref element="VT1" pad="3"/>
+<contactref element="R3" pad="2"/>
+<wire x1="67.31" y1="58.735" x2="67.63" y2="62.23" width="0" layer="19" extent="1-1"/>
+<wire x1="64.73" y1="59.42" x2="67.31" y2="58.735" width="0" layer="19" extent="1-1"/>
+<wire x1="59.69" y1="63.815" x2="64.73" y2="59.42" width="0" layer="19" extent="1-1"/>
+<wire x1="57.15" y1="62.865" x2="59.69" y2="63.815" width="0" layer="19" extent="1-1"/>
+<wire x1="54.61" y1="61.275" x2="57.15" y2="62.865" width="0" layer="19" extent="1-1"/>
+<wire x1="74.93" y1="54.61" x2="67.31" y2="58.735" width="0" layer="19" extent="1-1"/>
+</signal>
+<signal name="N$10">
+<contactref element="C3" pad="+"/>
+<contactref element="C3B" pad="1"/>
+<wire x1="44.135" y1="18.415" x2="44.45" y2="24.765" width="0" layer="19" extent="1-1"/>
+</signal>
 </signals>

Commit message: .
Parts:
- added D1, D2, D3: (no value), diode:SMC
- added U$1: (no value), B0_14CN3801:PCB1
- moved C1C 39.4 mm to (83.2, 43.8)
- moved C3B 33.7 mm to (73.7, 36.2)
- moved C3 30.6 mm to (71.1, 41.9)
- moved C1B 17.5 mm to (61.6, 43.8)
Other:
- board outline added: 120 x 120 mm
Changed lines of the file:
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@@
 <element name="VT1" library="m_transistor" package="TO220FV" value="" x="77.47" y="57.15" rot="R270"/>
 <element name="JP1" library="Разъёмы штырьковые 2.54мм" package="1X02" value="" x="57.15" y="61.595" rot="R270"/>
-<element name="C1B" library="rcl" package="C0805" value="1mf cer" x="45.085" y="38.1"/>
-<element name="C1C" library="rcl" package="E2,5-6" value="47m" x="45.72" y="31.75"/>
-<element name="C3" library="rcl" package="E2,5-6" value="10m louesr" x="45.72" y="24.765"/>
-<element name="C3B" library="rcl" package="C0805" value="1mf cer" x="45.085" y="18.415"/>
+<element name="C1B" library="rcl" package="C0805" value="1mf cer" x="61.595" y="43.815"/>
+<element name="C1C" library="rcl" package="E2,5-6" value="47m" x="83.185" y="43.815"/>
+<element name="C3" library="rcl" package="E2,5-6" value="10m louesr" x="71.12" y="41.91"/>
+<element name="C3B" library="rcl" package="C0805" value="1mf cer" x="73.66" y="36.195"/>
+<element name="D1" library="diode" package="SMC" value="" x="41.91" y="73.025"/>
+<element name="D2" library="diode" package="SMC" value="" x="42.545" y="60.325"/>
+<element name="D3" library="diode" package="SMC" value="" x="42.545" y="49.53"/>
+<element name="U$1" library="B0_14CN3801" package="PCB1" value="" x="51.435" y="39.37"/>
 </elements>
 <signals>
@@
 <wire x1="59.73" y1="59.42" x2="65.72" y2="54.61" width="0" layer="19" extent="1-1"/>
 <wire x1="57.15" y1="60.325" x2="59.73" y2="59.42" width="0" layer="19" extent="1-1"/>
-<wire x1="46.99" y1="24.765" x2="65.72" y2="54.61" width="0" layer="19" extent="1-1"/>
-<wire x1="46.035" y1="18.415" x2="46.99" y2="24.765" width="0" layer="19" extent="1-1"/>
+<wire x1="72.39" y1="41.91" x2="65.72" y2="54.61" width="0" layer="19" extent="1-1"/>
+<wire x1="74.61" y1="36.195" x2="72.39" y2="41.91" width="0" layer="19" extent="1-1"/>
 </signal>
 <signal name="N$5">
@@
 <contactref element="C3" pad="+"/>
 <contactref element="C3B" pad="1"/>
-<wire x1="44.135" y1="18.415" x2="44.45" y2="24.765" width="0" layer="19" extent="1-1"/>
+<wire x1="72.71" y1="36.195" x2="69.85" y2="41.91" width="0" layer="19" extent="1-1"/>
 </signal>
 </signals>

Commit message: .
Parts:
- added L1: (no value), rcl:PIS2816
- added L2: (no value), rcl:POWER-CHOKE_WE-TPC
- added L3: DR125, inductors:DR125
- added L4: DR127, inductors:DR127
- moved C2 2.62 mm to (62.2, 62.2), turned to 180 degrees
- moved C4 1.80 mm to (63.5, 53.3), turned to 90 degrees
- moved R2 1.42 mm to (61.0, 53.3), turned to 90 degrees
Connections:
- net N$4 renamed COM
Routing:
- net N$1: track 0.00 -> 15.4 mm
- net GND: track 0.00 -> 10.5 mm
- net N$5: track 0.00 -> 3.46 mm
- net COM: track 0.00 -> 2.64 mm
- net N$8: track 0.00 -> 2.54 mm
- net N$2: track 0.00 -> 2.49 mm
- net N$7: track 0.00 -> 1.94 mm
- net N$6: track 0.00 -> 1.83 mm
Changed lines of the file:
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@@
 <dimension x1="53.34" y1="44.45" x2="77.47" y2="41.275" x3="65.405" y3="76.835" textsize="1.778" layer="47" dtype="horizontal"/>
 <dimension x1="42.545" y1="65.405" x2="45.72" y2="51.435" x3="90.805" y3="58.42" textsize="1.778" layer="47" dtype="vertical"/>
+<dimension x1="43.18" y1="94.615" x2="55.88" y2="94.615" x3="49.53" y3="101.6" textsize="1.778" layer="1" dtype="horizontal"/>
+<dimension x1="76.2" y1="81.915" x2="83.82" y2="81.915" x3="80.01" y3="87.63" textsize="1.778" layer="1" dtype="horizontal"/>
 </plain>
 <attributes>
@@
 <elements>
 <element name="DA1" library="Consonance" package="SSOP10" value="CN3801" x="62.23" y="58.42"/>
-<element name="C2" library="rcl" package="C0805" value="100n" x="59.69" y="62.865" rot="R270"/>
+<element name="C2" library="rcl" package="C0805" value="100n" x="62.23" y="62.23" rot="R180"/>
 <element name="C1" library="rcl" package="C0805" value="100n" x="68.58" y="62.23"/>
 <element name="HL1" library="led" package="CHIPLED_0603" value="" x="57.15" y="58.42" rot="R270"/>
 <element name="HL2" library="led" package="CHIPLED_0603" value="" x="57.15" y="57.15" rot="R270"/>
 <element name="R1" library="rcl" package="R0805" value="" x="54.61" y="60.325" rot="R90"/>
-<element name="R2" library="rcl" package="R0805" value="120" x="60.325" y="54.61" rot="R180"/>
+<element name="R2" library="rcl" package="R0805" value="120" x="60.96" y="53.34" rot="R90"/>
 <element name="R3" library="rcl" package="R0805" value="" x="67.31" y="57.785" rot="R90"/>
 <element name="R4" library="rcl" package="R0805" value="" x="69.85" y="59.055" rot="R270"/>
-<element name="C4" library="rcl" package="C0805" value="220n" x="64.77" y="54.61"/>
+<element name="C4" library="rcl" package="C0805" value="220n" x="63.5" y="53.34" rot="R90"/>
 <element name="VT1" library="m_transistor" package="TO220FV" value="" x="77.47" y="57.15" rot="R270"/>
 <element name="JP1" library="Разъёмы штырьковые 2.54мм" package="1X02" value="" x="57.15" y="61.595" rot="R270"/>
@@
 <element name="D3" library="diode" package="SMC" value="" x="42.545" y="49.53"/>
 <element name="U$1" library="B0_14CN3801" package="PCB1" value="" x="51.435" y="39.37"/>
+<element name="L1" library="rcl" package="PIS2816" value="" x="80.01" y="78.74" rot="R90"/>
+<element name="L2" library="rcl" package="POWER-CHOKE_WE-TPC" value="" x="66.04" y="78.105" rot="R90"/>
+<element name="L3" library="inductors" package="DR125" value="DR125" x="49.53" y="87.63"/>
+<element name="L4" library="inductors" package="DR127" value="DR127" x="66.04" y="87.63"/>
 </elements>
 <signals>
@@
 <contactref element="DA1" pad="1"/>
 <contactref element="C2" pad="2"/>
-<wire x1="59.73" y1="60.42" x2="59.69" y2="61.915" width="0" layer="19" extent="1-1"/>
+<wire x1="59.69" y1="60.46" x2="59.73" y2="60.42" width="0.4064" layer="1"/>
+<wire x1="59.69" y1="60.46" x2="59.69" y2="60.64" width="0.4064" layer="1"/>
+<wire x1="59.69" y1="60.64" x2="61.28" y2="62.23" width="0.4064" layer="1"/>
 </signal>
 <signal name="GND">
@@
 <contactref element="C3" pad="-"/>
 <wire x1="69.85" y1="60.005" x2="69.53" y2="62.23" width="0" layer="19" extent="1-1"/>
-<wire x1="65.72" y1="54.61" x2="69.85" y2="60.005" width="0" layer="19" extent="1-1"/>
-<wire x1="59.73" y1="59.42" x2="65.72" y2="54.61" width="0" layer="19" extent="1-1"/>
-<wire x1="57.15" y1="60.325" x2="59.73" y2="59.42" width="0" layer="19" extent="1-1"/>
-<wire x1="72.39" y1="41.91" x2="65.72" y2="54.61" width="0" layer="19" extent="1-1"/>
+<wire x1="63.5" y1="54.29" x2="69.85" y2="60.005" width="0" layer="19" extent="1-1"/>
+<wire x1="72.39" y1="41.91" x2="63.5" y2="54.29" width="0" layer="19" extent="1-1"/>
 <wire x1="74.61" y1="36.195" x2="72.39" y2="41.91" width="0" layer="19" extent="1-1"/>
+<wire x1="59.73" y1="59.42" x2="61.23" y2="59.42" width="0.4064" layer="1"/>
+<wire x1="61.23" y1="59.42" x2="62.865" y2="57.785" width="0.4064" layer="1"/>
+<wire x1="62.865" y1="57.785" x2="62.865" y2="54.925" width="0.4064" layer="1"/>
+<wire x1="62.865" y1="54.925" x2="63.5" y2="54.29" width="0.4064" layer="1"/>
+<wire x1="59.73" y1="59.42" x2="58.055" y2="59.42" width="0.4064" layer="1"/>
+<wire x1="58.055" y1="59.42" x2="57.15" y2="60.325" width="0.4064" layer="1"/>
 </signal>
 <signal name="N$5">
@@
 <contactref element="HL2" pad="A"/>
 <contactref element="HL1" pad="A"/>
-<wire x1="56.4" y1="57.15" x2="56.4" y2="58.42" width="0" layer="19" extent="1-1"/>
-<wire x1="54.61" y1="59.375" x2="56.4" y2="58.42" width="0" layer="19" extent="1-1"/>
+<wire x1="56.4" y1="57.15" x2="56.4" y2="58.42" width="0.4064" layer="1"/>
+<wire x1="56.4" y1="58.42" x2="55.565" y2="58.42" width="0.4064" layer="1"/>
+<wire x1="55.565" y1="58.42" x2="54.61" y2="59.375" width="0.4064" layer="1"/>
 </signal>
 <signal name="N$6">
 <contactref element="HL1" pad="C"/>
 <contactref element="DA1" pad="3"/>
-<wire x1="57.9" y1="58.42" x2="59.73" y2="58.42" width="0" layer="19" extent="1-1"/>
+<wire x1="57.9" y1="58.42" x2="59.73" y2="58.42" width="0.4064" layer="1"/>
 </signal>
 <signal name="N$7">
 <contactref element="HL2" pad="C"/>
 <contactref element="DA1" pad="4"/>
-<wire x1="57.9" y1="57.15" x2="59.73" y2="57.42" width="0" layer="19" extent="1-1"/>
+<wire x1="59.73" y1="57.42" x2="58.17" y2="57.42" width="0.4064" layer="1"/>
+<wire x1="58.17" y1="57.42" x2="57.9" y2="57.15" width="0.4064" layer="1"/>
 </signal>
 <signal name="N$3">
@@
 <wire x1="64.73" y1="56.42" x2="67.31" y2="56.835" width="0" layer="19" extent="1-1"/>
 </signal>
-<signal name="N$4">
+<signal name="COM">
 <contactref element="DA1" pad="5"/>
 <contactref element="R2" pad="2"/>
-<wire x1="59.375" y1="54.61" x2="59.73" y2="56.42" width="0" layer="19" extent="1-1"/>
+<wire x1="59.73" y1="56.42" x2="59.73" y2="55.52" width="0.4064" layer="1"/>
+<wire x1="59.73" y1="55.52" x2="60.96" y2="54.29" width="0.4064" layer="1"/>
 </signal>
 <signal name="N$8">
 <contactref element="R2" pad="1"/>
 <contactref element="C4" pad="1"/>
-<wire x1="61.275" y1="54.61" x2="63.82" y2="54.61" width="0" layer="19" extent="1-1"/>
+<wire x1="60.96" y1="52.39" x2="63.5" y2="52.39" width="0.4064" layer="1"/>
 </signal>
 <signal name="N$9">
@@
 <wire x1="67.31" y1="58.735" x2="67.63" y2="62.23" width="0" layer="19" extent="1-1"/>
 <wire x1="64.73" y1="59.42" x2="67.31" y2="58.735" width="0" layer="19" extent="1-1"/>
-<wire x1="59.69" y1="63.815" x2="64.73" y2="59.42" width="0" layer="19" extent="1-1"/>
-<wire x1="57.15" y1="62.865" x2="59.69" y2="63.815" width="0" layer="19" extent="1-1"/>
-<wire x1="54.61" y1="61.275" x2="57.15" y2="62.865" width="0" layer="19" extent="1-1"/>
 <wire x1="74.93" y1="54.61" x2="67.31" y2="58.735" width="0" layer="19" extent="1-1"/>
+<wire x1="58.1" y1="63.815" x2="57.15" y2="62.865" width="0.4064" layer="1"/>
+<wire x1="57.15" y1="62.865" x2="55.245" y2="62.865" width="0.4064" layer="1"/>
+<wire x1="55.245" y1="62.865" x2="54.61" y2="62.23" width="0.4064" layer="1"/>
+<wire x1="54.61" y1="62.23" x2="54.61" y2="61.275" width="0.4064" layer="1"/>
+<wire x1="64.73" y1="59.42" x2="63.77" y2="59.42" width="0.4064" layer="1"/>
+<wire x1="63.18" y1="62.23" x2="63.18" y2="60.01" width="0.4064" layer="1"/>
+<wire x1="63.18" y1="60.01" x2="63.77" y2="59.42" width="0.4064" layer="1"/>
+<wire x1="58.1" y1="63.815" x2="62.55" y2="63.815" width="0.4064" layer="1"/>
+<wire x1="63.18" y1="62.23" x2="63.18" y2="63.185" width="0.4064" layer="1"/>
+<wire x1="63.18" y1="63.185" x2="62.55" y2="63.815" width="0.4064" layer="1"/>
 </signal>
 <signal name="N$10">

Commit message: .
Parts:
- removed L1: (no value), rcl:PIS2816
- removed L2: (no value), rcl:POWER-CHOKE_WE-TPC
- removed L4: DR127, inductors:DR127
- removed VT1: (no value), m_transistor:TO220FV
- added D4, D5, D6: (no value), diode:SMC
- added Q1, Q4: BSO201SP, transistor-fet:SO-8
- added Q2, Q3: BSS84, transistor-fet:SC75_INFINEON
- added R5: 332k, rcl:R0805
- added RSC: (no value), rcl:R0805
- added SJ1, SJ2: (no value), jumper:SJ
- R3: value (none) -> 43k
- R4: value (none) -> 15k
- moved D3 51.8 mm to (93.3, 59.7), turned to 270 degrees
- moved D1 46.4 mm to (86.4, 59.7), turned to 270 degrees
- moved L3 32.7 mm to (80.6, 77.5)
- moved U$1 18.2 mm to (42.5, 55.2)
- moved D2 9.03 mm to (36.8, 67.3), turned to 270 degrees
- moved C1 3.18 mm to (70.5, 59.7)
- moved R4 2.69 mm to (71.8, 57.1)
- moved R3 1.27 mm to (67.3, 56.5)
Connections:
- removed net N$10: C3.+, C3B.1
- new net BAT: DA1.7, Q3.2, SJ2.1
- new net CSP: DA1.8, Q2.2, SJ1.1
- new net N$11: L3.2, Q4.5, Q4.6, Q4.7, Q4.8
- new net N$12: Q2.1, Q3.1, Q4.4, R5.1
- new net N$13: D1.C, D3.C, D4.C, L3.1, Q1.5, Q1.6, Q1.7, Q1.8
- new net N$14: Q2.3, Q4.1, Q4.2, Q4.3, RSC.2, SJ1.2
- new net N$15: C3.+, C3B.1, Q3.3, R5.2, RSC.1, SJ2.2
- new net N$4: D2.A, D5.A, D6.A, JP1.1
- net GND: now also D1.A, D3.A, D4.A
- net N$1: now also D2.C, D5.C, D6.C, Q1.1, Q1.2, Q1.3; no longer JP1.1, VT1.3
- net N$9: now also Q1.4; no longer VT1.1
Routing:
- net N$1: track 15.4 -> 12.2 mm

Commit message: .
Parts:
- moved U$1 125.7 mm to (-83.2, 54.6)
- moved R4 5.85 mm to (67.3, 53.3), turned to 90 degrees
- moved SJ1 4.26 mm to (59.7, 69.8)
- moved Q2 4.07 mm to (64.1, 68.6)
- moved C1 3.24 mm to (69.8, 56.5), turned to 270 degrees
- moved Q3 2.62 mm to (71.8, 69.2)
- moved SJ2 2.01 mm to (74.3, 69.2)
- moved Q1 1.42 mm to (69.2, 64.8)
- moved R3 1.27 mm to (67.3, 57.8)
- moved L3 0.64 mm to (80.6, 76.8)
Connections:
- net GND: now also C1B.2, C1C.-
- net N$1: now also C1B.1, C1C.+

Commit message: .
Parts:
- moved C3B 47.4 mm to (95.9, 78.1), turned to 90 degrees
- moved C3 45.5 mm to (100.3, 76.8), turned to 90 degrees
- moved RSC 32.3 mm to (105.4, 74.3), turned to 270 degrees
- moved C1B 18.0 mm to (74.3, 56.5), turned to 270 degrees
- moved C1C 17.1 mm to (71.8, 56.5), turned to 270 degrees
- moved D3 9.03 mm to (100.3, 65.4)
- moved D1 6.84 mm to (92.7, 62.2)
- moved D4 5.46 mm to (82.5, 64.1)
- moved Q3 2.62 mm to (71.1, 71.8)
- moved SJ2 2.01 mm to (73.7, 71.1)
- moved R5 1.42 mm to (71.1, 74.9)
- moved L3 1.27 mm to (80.6, 78.1)

Commit message: эн
Parts:
- moved D6 15.1 mm to (36.8, 62.2), turned to 90 degrees
- moved D5 14.5 mm to (43.2, 62.2), turned to 90 degrees
- moved D2 14.3 mm to (50.2, 62.2), turned to 90 degrees
- moved SJ1 2.29 mm to (61.6, 68.6)
Routing:
- net N$1: track 12.2 -> 12.8 mm
Changed lines of the file:
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@@
 <element name="C3" library="rcl" package="E2,5-6" value="10m louesr" x="100.33" y="76.835" rot="R90"/>
 <element name="C3B" library="rcl" package="C0805" value="1mf cer" x="95.885" y="78.105" rot="R90"/>
-<element name="D2" library="diode" package="SMC" value="" x="36.83" y="67.31" rot="R270"/>
+<element name="D2" library="diode" package="SMC" value="" x="50.165" y="62.23" rot="R90"/>
 <element name="U$1" library="B0_14CN3801" package="PCB1" value="" x="-83.185" y="54.61"/>
 <element name="L3" library="inductors" package="DR125" value="DR125" x="80.645" y="78.105"/>
@@
 <element name="Q3" library="transistor-fet" package="SC75_INFINEON" value="BSS84" x="71.12" y="71.755"/>
 <element name="D4" library="diode" package="SMC" value="" x="82.55" y="64.135" rot="R270"/>
-<element name="D5" library="diode" package="SMC" value="" x="29.845" y="67.945" rot="R270"/>
-<element name="D6" library="diode" package="SMC" value="" x="22.86" y="67.945" rot="R270"/>
+<element name="D5" library="diode" package="SMC" value="" x="43.18" y="62.23" rot="R90"/>
+<element name="D6" library="diode" package="SMC" value="" x="36.83" y="62.23" rot="R90"/>
 <element name="D1" library="diode" package="SMC" value="" x="92.71" y="62.23" rot="R270"/>
 <element name="D3" library="diode" package="SMC" value="" x="100.33" y="65.405" rot="R270"/>
@@
 <element name="RSC" library="rcl" package="R0805" value="" x="105.41" y="74.295" rot="R270"/>
 <element name="R5" library="rcl" package="R0805" value="332k" x="71.12" y="74.93"/>
-<element name="SJ1" library="jumper" package="SJ" value="" x="59.69" y="69.85" rot="R270"/>
+<element name="SJ1" library="jumper" package="SJ" value="" x="61.595" y="68.58" rot="R270"/>
 <element name="SJ2" library="jumper" package="SJ" value="" x="73.66" y="71.12" rot="R270"/>
 </elements>
@@
 <wire x1="63.18" y1="62.23" x2="63.18" y2="60.01" width="0.4064" layer="1"/>
 <wire x1="63.18" y1="60.01" x2="63.77" y2="59.42" width="0.4064" layer="1"/>
-<wire x1="58.1" y1="63.815" x2="62.55" y2="63.815" width="0.4064" layer="1"/>
+<wire x1="57.465" y1="63.815" x2="62.55" y2="63.815" width="0.4064" layer="1"/>
 <wire x1="63.18" y1="62.23" x2="63.18" y2="63.185" width="0.4064" layer="1"/>
 <wire x1="63.18" y1="63.185" x2="62.55" y2="63.815" width="0.4064" layer="1"/>
@@
 <wire x1="66.4718" y1="64.135" x2="66.4718" y2="65.405" width="0" layer="19" extent="1-1"/>
 <wire x1="63.18" y1="63.185" x2="66.4718" y2="64.135" width="0" layer="19" extent="1-1"/>
+<wire x1="55.245" y1="62.865" x2="57.465" y2="63.815" width="0" layer="19" extent="1-1"/>
 <wire x1="67.31" y1="58.735" x2="64.73" y2="59.42" width="0" layer="19" extent="1-1"/>
 <wire x1="69.85" y1="57.465" x2="67.31" y2="58.735" width="0" layer="19" extent="1-1"/>
 <wire x1="71.755" y1="57.785" x2="69.85" y2="57.465" width="0" layer="19" extent="1-1"/>
 <wire x1="74.295" y1="57.465" x2="71.755" y2="57.785" width="0" layer="19" extent="1-1"/>
-<wire x1="55.245" y1="62.865" x2="58.1" y2="63.815" width="0" layer="19" extent="1-1"/>
-<wire x1="36.83" y1="71.01" x2="54.61" y2="62.23" width="0" layer="19" extent="1-1"/>
-<wire x1="29.845" y1="71.645" x2="36.83" y2="71.01" width="0" layer="19" extent="1-1"/>
-<wire x1="22.86" y1="71.645" x2="29.845" y2="71.645" width="0" layer="19" extent="1-1"/>
+<wire x1="50.165" y1="58.53" x2="54.61" y2="61.275" width="0" layer="19" extent="1-1"/>
+<wire x1="43.18" y1="58.53" x2="50.165" y2="58.53" width="0" layer="19" extent="1-1"/>
+<wire x1="36.83" y1="58.53" x2="43.18" y2="58.53" width="0" layer="19" extent="1-1"/>
 </signal>
 <signal name="CSP">
@@
 <contactref element="Q2" pad="2"/>
 <contactref element="SJ1" pad="1"/>
-<wire x1="59.69" y1="70.612" x2="64.135" y2="69.155" width="0" layer="19" extent="1-1"/>
+<wire x1="61.595" y1="69.342" x2="64.135" y2="69.155" width="0" layer="19" extent="1-1"/>
 <wire x1="64.73" y1="58.42" x2="64.135" y2="69.155" width="0" layer="19" extent="1-1"/>
 </signal>
@@
 <contactref element="D5" pad="A"/>
 <contactref element="D6" pad="A"/>
-<wire x1="36.83" y1="63.61" x2="57.15" y2="62.865" width="0" layer="19" extent="1-1"/>
-<wire x1="29.845" y1="64.245" x2="36.83" y2="63.61" width="0" layer="19" extent="1-1"/>
-<wire x1="22.86" y1="64.245" x2="29.845" y2="64.245" width="0" layer="19" extent="1-1"/>
+<wire x1="50.165" y1="65.93" x2="57.15" y2="62.865" width="0" layer="19" extent="1-1"/>
+<wire x1="43.18" y1="65.93" x2="50.165" y2="65.93" width="0" layer="19" extent="1-1"/>
+<wire x1="36.83" y1="65.93" x2="43.18" y2="65.93" width="0" layer="19" extent="1-1"/>
 </signal>
 <signal name="N$11">
@@
 <wire x1="86.7918" y1="69.85" x2="86.7918" y2="71.12" width="0" layer="19" extent="1-1"/>
 <wire x1="64.635" y1="68.005" x2="86.7918" y2="69.85" width="0" layer="19" extent="1-1"/>
-<wire x1="59.69" y1="69.088" x2="64.635" y2="68.005" width="0" layer="19" extent="1-1"/>
+<wire x1="61.595" y1="67.818" x2="64.635" y2="68.005" width="0" layer="19" extent="1-1"/>
 </signal>
 <signal name="N$15">
