File: B0_14CN3801.brd (EAGLE design)
At the start: 120 x 120 mm, 31 parts, among them Q1 BSO201SP, Q2 BSS84, Q3 BSS84, Q4 BSO201SP

Commit message: t
Parts:
- added D10, D11, D12, D13, D14, D15, D16, D17, D18, D19, D20, D7, D8, D9: (no value), diode:SMC
- added JP10, JP11: (no value), Разъёмы штырьковые 2.54мм:1X07
- added JP4: (no value), Разъёмы штырьковые 2.54мм:2X07
- added JP8, JP9: (no value), Разъёмы штырьковые 2.54мм:1X02
- added U$2, U$3: (no value), B0_14CN3801:T48K30
- added VT1, VT2: (no value), m_transistor:TO220BH
- moved U$1 191.8 mm to (67.9, 172.7)
Connections:
- new net N$10: D14.C, D7.C
- new net N$16: D13.C, D15.C
- new net N$17: D12.C, D16.C
- new net N$18: D11.C, D17.C
- new net N$19: D10.C, D18.C
- new net N$20: D19.C, D9.C
- new net N$21: D20.C, D8.C
Changed lines of the file:
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@@
 <setting verticaltext="up"/>
 </settings>
-<grid distance="25" unitdist="mil" unit="mil" style="lines" multiple="1" display="yes" altdistance="0.025" altunitdist="inch" altunit="inch"/>
+<grid distance="25" unitdist="mil" unit="mm" style="lines" multiple="1" display="yes" altdistance="0.025" altunitdist="inch" altunit="inch"/>
 <layers>
 <layer number="1" name="Top" color="4" fill="1" visible="yes" active="yes"/>
@@
 <dimension x1="40.64" y1="10.795" x2="101.6" y2="5.08" x3="71.12" y3="101.6" textsize="1.778" layer="1" dtype="horizontal"/>
 <dimension x1="19.05" y1="86.36" x2="12.065" y2="33.02" x3="114.935" y3="59.69" textsize="1.778" layer="21" dtype="vertical"/>
+<dimension x1="-108.585" y1="38.1" x2="-61.595" y2="37.465" x3="-85.09" y3="112.395" textsize="1.778" layer="21" dtype="horizontal"/>
+<dimension x1="-108.585" y1="116.205" x2="-12.065" y2="115.57" x3="-60.325" y3="125.73" textsize="1.778" layer="21" dtype="horizontal"/>
+<dimension x1="-59.055" y1="36.195" x2="-12.065" y2="35.56" x3="-35.56" y3="110.49" textsize="1.778" layer="21" dtype="horizontal"/>
 </plain>
 <attributes>
@@
 <element name="C3B" library="rcl" package="C0805" value="1mf cer" x="95.885" y="78.105" rot="R90"/>
 <element name="D2" library="diode" package="SMC" value="" x="50.165" y="62.23" rot="R90"/>
-<element name="U$1" library="B0_14CN3801" package="PCB1" value="" x="-83.185" y="54.61"/>
+<element name="U$1" library="B0_14CN3801" package="PCB1" value="" x="67.945" y="172.72"/>
 <element name="L3" library="inductors" package="DR125" value="DR125" x="80.645" y="78.105"/>
 <element name="Q1" library="transistor-fet" package="SO-8" value="BSO201SP" x="69.215" y="64.77"/>
@@
 <element name="SJ1" library="jumper" package="SJ" value="" x="61.595" y="68.58" rot="R270"/>
 <element name="SJ2" library="jumper" package="SJ" value="" x="73.66" y="71.12" rot="R270"/>
+<element name="JP4" library="Разъёмы штырьковые 2.54мм" package="2X07" value="" x="-125.73" y="38.1"/>
+<element name="JP8" library="Разъёмы штырьковые 2.54мм" package="1X02" value="" x="-92.075" y="93.345"/>
+<element name="JP9" library="Разъёмы штырьковые 2.54мм" package="1X02" value="" x="-80.645" y="93.98"/>
+<element name="U$2" library="B0_14CN3801" package="T48K30" value="" x="-85.09" y="67.31"/>
+<element name="U$3" library="B0_14CN3801" package="T48K30" value="" x="-35.56" y="66.675"/>
+<element name="VT1" library="m_transistor" package="TO220BH" value="" x="-92.075" y="103.505" rot="R90"/>
+<element name="VT2" library="m_transistor" package="TO220BH" value="" x="-66.675" y="103.505" rot="R90"/>
+<element name="D8" library="diode" package="SMC" value="" x="-98.425" y="40.64" rot="R180"/>
+<element name="D9" library="diode" package="SMC" value="" x="-98.425" y="47.625" rot="R180"/>
+<element name="D10" library="diode" package="SMC" value="" x="-98.425" y="54.61" rot="R180"/>
+<element name="D11" library="diode" package="SMC" value="" x="-98.425" y="61.595" rot="R180"/>
+<element name="D12" library="diode" package="SMC" value="" x="-98.425" y="68.58" rot="R180"/>
+<element name="D13" library="diode" package="SMC" value="" x="-98.425" y="75.565" rot="R180"/>
+<element name="D14" library="diode" package="SMC" value="" x="-98.425" y="82.55" rot="R180"/>
+<element name="D7" library="diode" package="SMC" value="" x="-71.755" y="82.55"/>
+<element name="D15" library="diode" package="SMC" value="" x="-71.755" y="75.565"/>
+<element name="D16" library="diode" package="SMC" value="" x="-71.755" y="68.58"/>
+<element name="D17" library="diode" package="SMC" value="" x="-71.755" y="61.595"/>
+<element name="D18" library="diode" package="SMC" value="" x="-71.755" y="54.61"/>
+<element name="D19" library="diode" package="SMC" value="" x="-71.755" y="47.625"/>
+<element name="D20" library="diode" package="SMC" value="" x="-71.755" y="40.64"/>
+<element name="JP10" library="Разъёмы штырьковые 2.54мм" package="1X07" value="" x="-107.315" y="46.99" rot="R90"/>
+<element name="JP11" library="Разъёмы штырьковые 2.54мм" package="1X07" value="" x="-99.695" y="3.81"/>
 </elements>
 <signals>
@@
 <wire x1="72.07" y1="74.93" x2="71.62" y2="71.18" width="0" layer="19" extent="1-1"/>
 </signal>
+<signal name="N$10">
+<contactref element="D14" pad="C"/>
+<contactref element="D7" pad="C"/>
+<wire x1="-75.455" y1="82.55" x2="-94.725" y2="82.55" width="0" layer="19" extent="1-1"/>
+</signal>
+<signal name="N$16">
+<contactref element="D13" pad="C"/>
+<contactref element="D15" pad="C"/>
+<wire x1="-75.455" y1="75.565" x2="-94.725" y2="75.565" width="0" layer="19" extent="1-1"/>
+</signal>
+<signal name="N$17">
+<contactref element="D12" pad="C"/>
+<contactref element="D16" pad="C"/>
+<wire x1="-75.455" y1="68.58" x2="-94.725" y2="68.58" width="0" layer="19" extent="1-1"/>
+</signal>
+<signal name="N$18">
+<contactref element="D11" pad="C"/>
+<contactref element="D17" pad="C"/>
+<wire x1="-75.455" y1="61.595" x2="-94.725" y2="61.595" width="0" layer="19" extent="1-1"/>
+</signal>
+<signal name="N$19">
+<contactref element="D10" pad="C"/>
+<contactref element="D18" pad="C"/>
+<wire x1="-75.455" y1="54.61" x2="-94.725" y2="54.61" width="0" layer="19" extent="1-1"/>
+</signal>
+<signal name="N$20">
+<contactref element="D9" pad="C"/>
+<contactref element="D19" pad="C"/>
+<wire x1="-75.455" y1="47.625" x2="-94.725" y2="47.625" width="0" layer="19" extent="1-1"/>
+</signal>
+<signal name="N$21">
+<contactref element="D8" pad="C"/>
+<contactref element="D20" pad="C"/>
+<wire x1="-75.455" y1="40.64" x2="-94.725" y2="40.64" width="0" layer="19" extent="1-1"/>
+</signal>
 </signals>

Commit message: .
Parts:
- added JP2, JP3: (no value), Разъёмы штырьковые 2.54мм:1X02
- moved D7 82.7 mm to (-105.4, 6.99), turned to 90 degrees
- moved D14 79.7 mm to (-105.4, 3.17), flipped to the bottom, turned to 90 degrees
- moved D15 73.6 mm to (-98.4, 6.99), turned to 90 degrees
- moved D13 72.4 mm to (-98.4, 3.17), flipped to the bottom, turned to 90 degrees
- moved D12 65.8 mm to (-91.4, 3.17), flipped to the bottom, turned to 90 degrees
- moved D16 64.7 mm to (-91.4, 6.99), turned to 90 degrees
- moved D11 60.1 mm to (-84.5, 3.17), flipped to the bottom, turned to 90 degrees
- moved D17 56.1 mm to (-84.5, 6.99), turned to 90 degrees
- moved D10 55.5 mm to (-77.5, 3.17), flipped to the bottom, turned to 90 degrees
- moved D9 53.2 mm to (-69.2, 3.17), flipped to the bottom, turned to 90 degrees
- moved D8 51.2 mm to (-63.5, 3.17), flipped to the bottom, turned to 90 degrees
- moved D18 48.0 mm to (-77.5, 6.99), turned to 90 degrees
- moved D19 40.7 mm to (-70.5, 6.99), turned to 90 degrees
- moved D20 34.7 mm to (-63.5, 6.99), turned to 90 degrees
- moved JP11 19.7 mm to (-83.2, -6.99), turned to 180 degrees
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Connections:
- new net N$22: D19.A, JP3.2
- new net N$23: D9.A, JP3.1
- new net N$24: D8.A, JP2.1
- new net N$25: D20.A, JP2.2
- net N$10: now also JP11.7
- net N$16: now also JP11.6
- net N$17: now also JP11.5
- net N$18: now also JP11.4
- net N$19: now also JP11.3
- net N$20: now also JP11.2
- net N$21: now also JP11.1
Routing:
- net N$24: track 0.00 -> 8.89 mm
- net N$23: track 0.00 -> 8.37 mm
- net N$25: track 0.00 -> 5.08 mm
- net N$22: track 0.00 -> 5.08 mm
